File: OpenCoffee_PCB/OpenCoffeePCB/OpenCoffeePCB.kicad_sch (KiCad schematic)
At the start: 1 part, among them U1 Pico

Commit message: updates pcb
Parts:
- added J?: Conn_01x02_Male, symbol Connector:Conn_01x02_Male
- added U2: Pico_WiFi, MCU_RaspberryPi_and_Boards:RPi_Pico_SMD_TH_WIFI, symbol MCU_RaspberryPi_and_Boards:Pico_WiFi
Connections:
- net Button: now reaches U1.1 (GPIO0)
- net Display_SCL: now reaches U1.10 (GPIO7)
- net UART_TX: now reaches U1.11 (GPIO8)
- net UART_RX: now reaches U1.12 (GPIO9)
- net GroupHeadSolenoid: now reaches U1.17 (GPIO13)
- net Rotary_DT: now reaches U1.2 (GPIO1)
- net MAX6675_SCK: now reaches U1.20 (GPIO15)
- net MAX6675_CS: now reaches U1.21 (GPIO16)
- net MAX6675_SO: now reaches U1.22 (GPIO17)
- net DimmerPWM: now reaches U1.24 (GPIO18)
- net PressureSDA: now reaches U1.26 (GPIO20)
- net PressureSCL: now reaches U1.27 (GPIO21)
- net Heater: now reaches U1.31 (GPIO26_ADC0)
- net Rotary_CLK: now reaches U1.4 (GPIO2)
- net Display_SDA: now reaches U1.9 (GPIO6)
Other:
- moved on the sheet: U1
Changed lines of the file:
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@@
 (kicad_sch (version 20211123) (generator eeschema)
   (paper "A4")
-  (symbol (lib_id "MCU_RaspberryPi_and_Boards:Pico") (at 129.54 110.49 0) (unit 1)
+  (global_label "UART_RX" (shape input) (at 85.09 113.03 180) (fields_autoplaced)
+    (effects (font (size 1.27 1.27)) (justify right))
+    (property "Intersheet References" "${INTERSHEET_REFS}" (id 0) (at 74.5731 112.9506 0)
+      (effects (font (size 1.27 1.27)) (justify right) hide)
+    )
+  )
+  (global_label "MAX6675_SO" (shape input) (at 120.65 130.81 0) (fields_autoplaced)
+    (effects (font (size 1.27 1.27)) (justify left))
+    (property "Intersheet References" "${INTERSHEET_REFS}" (id 0) (at 135.1583 130.7306 0)
+      (effects (font (size 1.27 1.27)) (justify left) hide)
+    )
+  )
+  (global_label "Rotary_DT" (shape input) (at 85.09 87.63 180) (fields_autoplaced)
+    (effects (font (size 1.27 1.27)) (justify right))
+    (property "Intersheet References" "${INTERSHEET_REFS}" (id 0) (at 73.424 87.5506 0)
+      (effects (font (size 1.27 1.27)) (justify right) hide)
+    )
+  )
+  (global_label "UART_TX" (shape input) (at 85.09 110.49 180) (fields_autoplaced)
+    (effects (font (size 1.27 1.27)) (justify right))
+    (property "Intersheet References" "${INTERSHEET_REFS}" (id 0) (at 74.8755 110.4106 0)
+      (effects (font (size 1.27 1.27)) (justify right) hide)
+    )
+  )
+  (global_label "PressureSCL" (shape input) (at 120.65 118.11 0) (fields_autoplaced)
+    (effects (font (size 1.27 1.27)) (justify left))
+    (property "Intersheet References" "${INTERSHEET_REFS}" (id 0) (at 134.7955 118.0306 0)
+      (effects (font (size 1.27 1.27)) (justify left) hide)
+    )
+  )
+  (global_label "MAX6675_CS" (shape input) (at 120.65 133.35 0) (fields_autoplaced)
+    (effects (font (size 1.27 1.27)) (justify left))
+    (property "Intersheet References" "${INTERSHEET_REFS}" (id 0) (at 135.0979 133.4294 0)
+      (effects (font (size 1.27 1.27)) (justify left) hide)
+    )
+  )
+  (global_label "MAX6675_SCK" (shape input) (at 85.09 133.35 180) (fields_autoplaced)
+    (effects (font (size 1.27 1.27)) (justify right))
+    (property "Intersheet References" "${INTERSHEET_REFS}" (id 0) (at 69.3721 133.2706 0)
+      (effects (font (size 1.27 1.27)) (justify right) hide)
+    )
+  )
+  (global_label "Rotary_CLK" (shape input) (at 85.09 92.71 180) (fields_autoplaced)
+    (effects (font (size 1.27 1.27)) (justify right))
+    (property "Intersheet References" "${INTERSHEET_REFS}" (id 0) (at 72.0936 92.6306 0)
+      (effects (font (size 1.27 1.27)) (justify right) hide)
+    )
+  )
+  (global_label "PressureSDA" (shape input) (at 120.65 120.65 0) (fields_autoplaced)
+    (effects (font (size 1.27 1.27)) (justify left))
+    (property "Intersheet References" "${INTERSHEET_REFS}" (id 0) (at 134.856 120.5706 0)
+      (effects (font (size 1.27 1.27)) (justify left) hide)
+    )
+  )
+  (global_label "Button" (shape input) (at 85.09 85.09 180) (fields_autoplaced)
+    (effects (font (size 1.27 1.27)) (justify right))
+    (property "Intersheet References" "${INTERSHEET_REFS}" (id 0) (at 76.5083 85.0106 0)
+      (effects (font (size 1.27 1.27)) (justify right) hide)
+    )
+  )
+  (global_label "Display_SCL" (shape input) (at 85.09 107.95 180) (fields_autoplaced)
+    (effects (font (size 1.27 1.27)) (justify right))
+    (property "Intersheet References" "${INTERSHEET_REFS}" (id 0) (at 71.3679 107.8706 0)
+      (effects (font (size 1.27 1.27)) (justify right) hide)
+    )
+  )
+  (global_label "Display_SDA" (shape input) (at 85.09 105.41 180) (fields_autoplaced)
+    (effects (font (size 1.27 1.27)) (justify right))
+    (property "Intersheet References" "${INTERSHEET_REFS}" (id 0) (at 71.3074 105.3306 0)
+      (effects (font (size 1.27 1.27)) (justify right) hide)
+    )
+  )
+  (hierarchical_label "GroupHeadSolenoid" (shape input) (at 85.09 125.73 180)
+    (effects (font (size 1.27 1.27)) (justify right))
+  )
+  (hierarchical_label "Heater" (shape input) (at 120.65 107.95 0)
+    (effects (font (size 1.27 1.27)) (justify left))
+  )
+  (hierarchical_label "DimmerPWM" (shape input) (at 120.65 125.73 0)
+    (effects (font (size 1.27 1.27)) (justify left))
+  )
+  (symbol (lib_id "Connector:Conn_01x02_Male") (at 33.02 134.62 0) (unit 1)
     (in_bom yes) (on_board yes) (fields_autoplaced)
-    (property "Reference" "U1" (id 0) (at 129.54 78.74 0))
-    (property "Value" "Pico" (id 1) (at 129.54 81.28 0))
-    (property "Footprint" "MCU_RaspberryPi_and_Boards:RPi_Pico_SMD_TH" (id 2) (at 129.54 110.49 90)
-      (effects (font (size 1.27 1.27)) hide)
-    )
-    (property "Datasheet" "" (id 3) (at 129.54 110.49 0)
+    (property "Reference" "J?" (id 0) (at 33.655 129.54 0))
+    (property "Value" "Conn_01x02_Male" (id 1) (at 33.655 132.08 0))
+    (property "Footprint" "" (id 2) (at 33.02 134.62 0)
+      (effects (font (size 1.27 1.27)) hide)
+    )
+    (property "Datasheet" "~" (id 3) (at 33.02 134.62 0)
+      (effects (font (size 1.27 1.27)) hide)
+    )
+    (pin "1")
+    (pin "2")
+  )
+  (symbol (lib_id "MCU_RaspberryPi_and_Boards:Pico") (at 102.87 109.22 0) (unit 1)
+    (in_bom yes) (on_board yes) (fields_autoplaced)
+    (property "Reference" "U1" (id 0) (at 102.87 77.47 0))
+    (property "Value" "Pico" (id 1) (at 102.87 80.01 0))
+    (property "Footprint" "MCU_RaspberryPi_and_Boards:RPi_Pico_SMD_TH" (id 2) (at 102.87 109.22 90)
+      (effects (font (size 1.27 1.27)) hide)
+    )
+    (property "Datasheet" "" (id 3) (at 102.87 109.22 0)
       (effects (font (size 1.27 1.27)) hide)
     )
@@
     (pin "9")
   )
+  (symbol (lib_id "MCU_RaspberryPi_and_Boards:Pico_WiFi") (at 182.88 111.76 0) (unit 1)
+    (in_bom yes) (on_board yes) (fields_autoplaced)
+    (property "Reference" "U2" (id 0) (at 182.88 80.01 0))
+    (property "Value" "Pico_WiFi" (id 1) (at 182.88 82.55 0))
+    (property "Footprint" "MCU_RaspberryPi_and_Boards:RPi_Pico_SMD_TH_WIFI" (id 2) (at 182.88 111.76 90)
+      (effects (font (size 1.27 1.27)) hide)
+    )
+    (property "Datasheet" "" (id 3) (at 182.88 111.76 0)
+      (effects (font (size 1.27 1.27)) hide)
+    )
+    (pin "1")
+    (pin "10")
+    (pin "11")
+    (pin "12")
+    (pin "13")
+    (pin "14")
+    (pin "15")
+    (pin "16")
+    (pin "17")
+    (pin "18")
+    (pin "19")
+    (pin "2")
+    (pin "20")
+    (pin "21")
+    (pin "22")
+    (pin "23")
+    (pin "24")
+    (pin "25")
+    (pin "26")
+    (pin "27")
+    (pin "28")
+    (pin "29")
+    (pin "3")
+    (pin "30")
+    (pin "31")
+    (pin "32")
+    (pin "33")
+    (pin "34")
+    (pin "35")
+    (pin "36")
+    (pin "37")
+    (pin "38")
+    (pin "39")
+    (pin "4")
+    (pin "40")
+    (pin "41")
+    (pin "42")
+    (pin "43")
+    (pin "5")
+    (pin "6")
+    (pin "7")
+    (pin "8")
+    (pin "9")
+  )
   (sheet_instances
     (path "/" (page "1"))
   )
   (symbol_instances
+    (path "/3d4cfd87-40bf-404a-939f-7f1a4bb9f65b"
+      (reference "J?") (unit 1) (value "Conn_01x02_Male") (footprint "")
+    )
     (path "/a1a26910-ad02-491b-87ba-b3ce2db8ff52"
       (reference "U1") (unit 1) (value "Pico") (footprint "MCU_RaspberryPi_and_Boards:RPi_Pico_SMD_TH")
     )
-  )
+    (path "/a23dc7d1-f994-4417-a95d-774b11f1abab"
+      (reference "U2") (unit 1) (value "Pico_WiFi") (footprint "MCU_RaspberryPi_and_Boards:RPi_Pico_SMD_TH_WIFI")
+    )
+  )
