File: OpenCoffee_PCB/OpenCoffeePCB/OpenCoffeePCB.kicad_sch (KiCad schematic)
At the start: 3 parts, among them U1 Pico, U2 Pico_WiFi

Commit message: intial layout
Parts:
- removed J?: Conn_01x02_Male, symbol Connector:Conn_01x02_Male
- added J1, J2, J3, J4, J5: Conn_01x02_Male, Connector_Molex:Molex_KK-254_AE-6410-03A_1x03_P2.54mm_Vertical, symbol Connector:Conn_01x02_Male
- added J6, J7: Conn_01x03_Male, Connector_Molex:Molex_KK-254_AE-6410-03A_1x03_P2.54mm_Vertical, symbol Connector:Conn_01x03_Male
- added J8: Barrel_Jack_Switch, Connector_BarrelJack:BarrelJack_GCT_DCJ200-10-A_Horizontal, symbol Connector:Barrel_Jack_Switch
Connections:
- net DimmerPWM: now also J2.2 (Pin_2)
- net Display_SCL: now also J3.1 (Pin_1)
- net Display_SDA: now also J3.2 (Pin_2)
- net GroupHeadSolenoid: now also J5.2 (Pin_2)
- net Heater: now also J5.1 (Pin_1)
- net MAX6675_CS: now also J6.3 (Pin_3)
- net MAX6675_SCK: now also J6.1 (Pin_1)
- net MAX6675_SO: now also J6.2 (Pin_2)
- net PressureSCL: now also J1.1 (Pin_1)
- net PressureSDA: now also J1.2 (Pin_2)
- net Rotary_CLK: now also J7.1 (Pin_1)
- net Rotary_DT: now also J7.2 (Pin_2)
- net UART_RX: now also U2.4 (GPIO2), J4.1 (Pin_1)
- net UART_TX: now also U2.5 (GPIO3), J4.2 (Pin_2)
- net GND: now reaches U1.28 (GND)
- net GND: now also U2.28 (GND), J8.2, J8.3
- net 5V: now reaches U1.36 (3V3)
- net 5V: now also U2.36 (3V3), J8.1
- net Button renamed Rotary_Button
- net Rotary_Button: now also J7.3 (Pin_3)

Commit message: working on max6675
Parts:
- added U3: MAX6675, OpenCoffeePartsFootprint:MAX6675, symbol OpenCoffeeParts:MAX6675
Connections:
- net GND: now also U3.1 (GND)
Changed lines of the file:
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@@
+    )
+  )
+  (global_label "GND" (shape input) (at 246.38 107.95 0) (fields_autoplaced)
+    (effects (font (size 1.27 1.27)) (justify left))
+    (property "Intersheet References" "${INTERSHEET_REFS}" (id 0) (at 252.6636 107.8706 0)
+      (effects (font (size 1.27 1.27)) (justify left) hide)
     )
   )
@@
       (effects (font (size 1.27 1.27)) (justify right) hide)
     )
+  )
+  (symbol (lib_id "OpenCoffeeParts:MAX6675") (at 256.54 100.33 0) (unit 1)
+    (in_bom yes) (on_board yes) (fields_autoplaced)
+    (property "Reference" "U3" (id 0) (at 238.2394 100.33 0)
+      (effects (font (size 1.27 1.27)) (justify left))
+    )
+    (property "Value" "MAX6675" (id 1) (at 238.2394 102.87 0)
+      (effects (font (size 1.27 1.27)) (justify left))
+    )
+    (property "Footprint" "OpenCoffeePartsFootprint:MAX6675" (id 2) (at 256.54 100.33 0)
+      (effects (font (size 1.27 1.27)) hide)
+    )
+    (property "Datasheet" "" (id 3) (at 256.54 100.33 0)
+      (effects (font (size 1.27 1.27)) hide)
+    )
+    (pin "1")
+    (pin "2")
+    (pin "3")
+    (pin "4")
+    (pin "5")
+    (pin "6")
+    (pin "7")
+    (pin "8")
   )
   (symbol (lib_id "Connector:Conn_01x02_Male") (at 50.8 109.22 180) (unit 1)
@@
       (reference "U2") (unit 1) (value "Pico_WiFi") (footprint "MCU_RaspberryPi_and_Boards:RPi_Pico_SMD_TH_WIFI")
     )
-  )
+    (path "/20a43104-38cb-4a67-8590-5917234169dc"
+      (reference "U3") (unit 1) (value "MAX6675") (footprint "OpenCoffeePartsFootprint:MAX6675")
+    )
+  )

Commit message: working on pcb
Parts:
- added C1: 0.1uF, Capacitor_SMD:C_0805_2012Metric, symbol Device:C
- added J9: Conn_01x02_Male, Connector_Molex:Molex_KK-254_AE-6410-02A_1x02_P2.54mm_Vertical, symbol Connector:Conn_01x02_Male
- J1, J2, J3, J4, J5: footprint Connector_Molex:Molex_KK-254_AE-6410-03A_1x03_P2.54mm_Vertical -> Connector_Molex:Molex_KK-254_AE-6410-02A_1x02_P2.54mm_Vertical
Connections:
- net 5V: now also U1.39 (VSYS), U2.39 (VSYS), U3.4 (VCC), C1.1; no longer U1.36 (3V3), U2.36 (3V3)
- net GND: now also C1.2
- net MAX6675_CS: now also U3.6 (CS)
- net MAX6675_SCK: now also U3.5 (SCK)
- net MAX6675_SO: now also U3.7 (SO)
- net T-: now reaches U3.2 (T-)
- net T-: now also J9.1 (Pin_1)
- net T+: now reaches U3.3 (T+)
- net T+: now also J9.2 (Pin_2)
- no-connect marks 0 -> 1

Commit message: making PCB
Parts:
- added J10: Conn_01x02_Male, Connector_Molex:Molex_KK-254_AE-6410-02A_1x02_P2.54mm_Vertical, symbol Connector:Conn_01x02_Male
Connections:
- net GND: now also U1.13 (GND), U1.18 (GND), U1.23 (GND), U1.42 (GND), U2.13 (GND), U2.18 (GND), U2.23 (GND), U2.3 (GND), U2.33 (AGND), U2.38 (GND), U2.8 (GND)
- net UART_RX: now also J10.1 (Pin_1); no longer J4.1 (Pin_1), U2.4 (GPIO2)
- net UART_TX: now also J10.2 (Pin_2); no longer J4.2 (Pin_2), U2.5 (GPIO3)
- new net UART_RX_W: J4.1 (Pin_1), U2.4 (GPIO2)
- new net UART_TX_W: J4.2 (Pin_2), U2.5 (GPIO3)
- no-connect marks 1 -> 56
Other:
- moved on the sheet: J4

Commit message: part
Parts:
- C1: value 0.1uF -> C
Changed lines of the file:
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@@
       (effects (font (size 1.27 1.27)) (justify left))
     )
-    (property "Value" "0.1uF" (at 240.03 128.905 0)
+    (property "Value" "C" (at 240.03 128.905 0)
       (effects (font (size 1.27 1.27)) (justify left))
     )
@@
       (effects (font (size 1.27 1.27)) hide)
     )
-    (property "Datasheet" "C28233" (at 236.22 127 0)
+    (property "Datasheet" "~" (at 236.22 127 0)
       (effects (font (size 1.27 1.27)) hide)
     )
@@
       (effects (font (size 1.27 1.27)) hide)
     )
-    (property "Datasheet" "C319098" (at 156.21 65.786 0)
+    (property "Datasheet" "~" (at 156.21 65.786 0)
       (effects (font (size 1.27 1.27)) hide)
     )
