File: OpenCoffee_PCB/OpenCoffeePCB/OpenCoffeePCB.kicad_sch (KiCad schematic)
At the start: 14 parts, among them J1 Conn_01x02_Male, J10 Conn_01x02_Male, J2 Conn_01x02_Male, J3 Conn_01x02_Male, J4 Conn_01x02_Male, J5 Conn_01x02_Male, J6 Conn_01x03_Male, J7 Conn_01x03_Male, J8 Barrel_Jack_Switch, J9 Conn_01x02_Male, U1 Pico, U2 Pico_WiFi, U3 MAX6675

Commit message: added RP2040 from https://datasheets.raspberrypi.com/rp2040/Minimal-KiCAD.zip?_gl=1*n2lfxt*_ga*MTI3MDcyNzk1MS4xNjg5NTU4NDUx*_ga_22FD70LWDS*MTY4OTU1ODQ1Mi4xLjEuMTY4OTU1OTgzMS4wLjAuMA..
Parts:
- added C10, C12, C13, C14, C15, C16, C17, C4, C7, C8: 100n, Capacitor_SMD:C_0402_1005Metric, symbol Device:C
- added C11, C9: 1u, Capacitor_SMD:C_0402_1005Metric, symbol Device:C
- added C2, C3: 10u, Capacitor_SMD:C_0805_2012Metric, symbol Device:C
- added C5, C6: 27p, Capacitor_SMD:C_0402_1005Metric, symbol Device:C
- added J11: USB_B_Micro, RP2040_minimal:USB_Micro-B_Amphenol_10103594-0001LF_Horizontal_modified, symbol RP2040_minimal-rescue:USB_B_Micro-Connector
- added J12: Conn_01x02, Connector_PinHeader_2.54mm:PinHeader_1x02_P2.54mm_Vertical, symbol Connector_Generic:Conn_01x02
- added R1, R3: 1k, Capacitor_SMD:C_0402_1005Metric, symbol Device:R
- added R2: DNF, Capacitor_SMD:C_0402_1005Metric, symbol Device:R
- added R4, R5: 27, Capacitor_SMD:C_0402_1005Metric, symbol Device:R
- added U4: NCP1117-3.3_SOT223, Package_TO_SOT_SMD:SOT-223-3_TabPin2, symbol Regulator_Linear:NCP1117-3.3_SOT223
- added U5: W25Q128JVS, Package_SO:SOIC-8_5.23x5.23mm_P1.27mm, symbol RP2040_minimal-rescue:W25Q128JVS-Memory_Flash
- added U6: RP2040, RP2040_minimal:RP2040-QFN-56, symbol RP2040_minimal-rescue:RP2040-MCU_RaspberryPi_RP2040
- added Y1: ABLS-12.000MHZ-B4-T, RP2040_minimal:Crystal_SMD_HC49-US, symbol Device:Crystal
Connections:
- net GND: now also C10.2, C11.2, C12.2, C13.2, C14.2, C15.2, C16.2, C17.2, C2.2, C3.2, C4.2, C5.2, C6.2, C7.2, C8.2, C9.2, J11.5 (GND), J11.6 (Shield), J12.2 (Pin_2), U4.1 (GND), U5.4 (GND), U6.19 (TESTEN), U6.57 (GND)
- new net: R5.2, U6.46 (USB_DM)
- new net: R4.2, U6.47 (USB_DP)
- new net: C6.1, R3.2, Y1.2
- new net +1V1: C7.1, C8.1, C9.1, U6.23 (DVDD), U6.45 (VREG_VOUT), U6.50 (DVDD)
- new net +3V3: C10.1, C11.1, C12.1, C13.1, C14.1, C15.1, C16.1, C17.1, C3.1, C4.1, R2.1, U4.2 (VO), U5.8 (VCC), U6.1 (IOVDD), U6.10 (IOVDD), U6.22 (IOVDD), U6.33 (IOVDD), U6.42 (IOVDD), U6.43 (ADC_AVDD), U6.44 (VREG_IN), U6.48 (USB_VDD), U6.49 (IOVDD)
- new net GPIO0: U6.2 (GPIO0)
- new net GPIO1: U6.3 (GPIO1)
- new net GPIO10: U6.13 (GPIO10)
- new net GPIO11: U6.14 (GPIO11)
- new net GPIO12: U6.15 (GPIO12)
- new net GPIO13: U6.16 (GPIO13)
- new net GPIO14: U6.17 (GPIO14)
- new net GPIO15: U6.18 (GPIO15)
- new net GPIO16: U6.27 (GPIO16)
- new net GPIO17: U6.28 (GPIO17)
- new net GPIO18: U6.29 (GPIO18)
- new net GPIO19: U6.30 (GPIO19)
- new net GPIO2: U6.4 (GPIO2)
- new net GPIO20: U6.31 (GPIO20)
- new net GPIO21: U6.32 (GPIO21)
- new net GPIO22: U6.34 (GPIO22)
- new net GPIO23: U6.35 (GPIO23)
- new net GPIO24: U6.36 (GPIO24)
- new net GPIO25: U6.37 (GPIO25)
- new net GPIO26_ADC0: U6.38 (GPIO26_ADC0)
- new net GPIO27_ADC1: U6.39 (GPIO27_ADC1)
- new net GPIO28_ADC2: U6.40 (GPIO28_ADC2)
- new net GPIO29_ADC3: U6.41 (GPIO29_ADC3)
- new net GPIO3: U6.5 (GPIO3)
- new net GPIO4: U6.6 (GPIO4)
- new net GPIO5: U6.7 (GPIO5)
- new net GPIO6: U6.8 (GPIO6)
- new net GPIO7: U6.9 (GPIO7)
- new net GPIO8: U6.11 (GPIO8)
- new net GPIO9: U6.12 (GPIO9)
- new net QSPI_SCLK: U5.6 (CLK), U6.52 (QSPI_SCLK)
- new net QSPI_SD0: U5.5 (DI(IO0)), U6.53 (QSPI_SD0)
- new net QSPI_SD1: U5.2 (DO(IO1)), U6.55 (QSPI_SD1)
- new net QSPI_SD2: U5.3 (IO2), U6.54 (QSPI_SD2)
- new net QSPI_SD3: U5.7 (IO3), U6.51 (QSPI_SD3)
- new net QSPI_SS: R1.1, R2.2, U5.1 (~{CS}), U6.56 (QSPI_SS)
- new net RUN: U6.26 (RUN)
- new net SWCLK: U6.24 (SWCLK)
- new net SWD: U6.25 (SWD)
- new net USB_D+: J11.3 (D+), R4.1
- new net USB_D-: J11.2 (D-), R5.1
- new net VBUS: C2.1, J11.1 (VBUS), U4.3 (VI)
- new net XIN: C5.1, U6.20 (XIN), Y1.1
- new net XOUT: R3.1, U6.21 (XOUT)
- new net ~{USB_BOOT}: J12.1 (Pin_1), R1.2
- no-connect marks 56 -> 57
Other:
- note added: "Crystal"
- note added: "Flash"
- note added: "Make sure C10 is close to pin 44 of RP2040"
- note added: "Make sure C8 is close to pin 45 of RP2040"
- note added: "Make sure R3 and R4 are close to RP2040"
- note added: "Power"
