File: OpenCoffee_PCB/OpenCoffeePCB/OpenCoffeePCB.kicad_pcb (KiCad board)
At the start: 2 copper layers, 1 part, among them U1 Pico

Commit message: updates pcb
Parts:
- added U2: Pico_WiFi, MCU_RaspberryPi_and_Boards:RPi_Pico_SMD_TH_WIFI, F.Cu at (167.6, 66.0)

Commit message: intial layout
Parts:
- added J1: Conn_01x02_Male, Connector_Molex:Molex_KK-254_AE-6410-03A_1x03_P2.54mm_Vertical, F.Cu at (111.8, 91.4)
- added J2: Conn_01x02_Male, Connector_Molex:Molex_KK-254_AE-6410-03A_1x03_P2.54mm_Vertical, F.Cu at (111.8, 55.9)
- added J3: Conn_01x02_Male, Connector_Molex:Molex_KK-254_AE-6410-03A_1x03_P2.54mm_Vertical, F.Cu at (121.9, 99.1)
- added J4: Conn_01x02_Male, Connector_Molex:Molex_KK-254_AE-6410-03A_1x03_P2.54mm_Vertical, F.Cu at (111.8, 45.7)
- added J5: Conn_01x02_Male, Connector_Molex:Molex_KK-254_AE-6410-03A_1x03_P2.54mm_Vertical, F.Cu at (111.8, 78.7)
- added J6: Conn_01x03_Male, Connector_Molex:Molex_KK-254_AE-6410-03A_1x03_P2.54mm_Vertical, F.Cu at (134.6, 99.1)
- added J7: Conn_01x03_Male, Connector_Molex:Molex_KK-254_AE-6410-03A_1x03_P2.54mm_Vertical, F.Cu at (111.8, 68.6)
- added J8: Barrel_Jack_Switch, Connector_BarrelJack:BarrelJack_GCT_DCJ200-10-A_Horizontal, F.Cu at (185.4, 53.3)
- moved U1 10.2 mm to (134.6, 66.0)
- moved U2 2.54 mm to (165.1, 66.0)
Connections:
- U1 pad 1: unconnected-(U1-Pad1) -> Rotary_Button
- U1 pad 10: unconnected-(U1-Pad10) -> Display_SCL
- U1 pad 11: unconnected-(U1-Pad11) -> UART_TX
- U1 pad 12: unconnected-(U1-Pad12) -> UART_RX
- U1 pad 17: unconnected-(U1-Pad17) -> GroupHeadSolenoid
- U1 pad 2: unconnected-(U1-Pad2) -> Rotary_DT
- U1 pad 20: unconnected-(U1-Pad20) -> MAX6675_SCK
- U1 pad 21: unconnected-(U1-Pad21) -> MAX6675_CS
- U1 pad 22: unconnected-(U1-Pad22) -> MAX6675_SO
- U1 pad 24: unconnected-(U1-Pad24) -> DimmerPWM
- U1 pad 26: unconnected-(U1-Pad26) -> PressureSDA
- U1 pad 27: unconnected-(U1-Pad27) -> PressureSCL
- U1 pad 28: unconnected-(U1-Pad28) -> GND
- U1 pad 31: unconnected-(U1-Pad31) -> Heater
- U1 pad 36: unconnected-(U1-Pad36) -> 5V
- U1 pad 4: unconnected-(U1-Pad4) -> Rotary_CLK
- U1 pad 9: unconnected-(U1-Pad9) -> Display_SDA
- U2 pad 28: unconnected-(U2-Pad28) -> GND
- U2 pad 36: unconnected-(U2-Pad36) -> 5V
- U2 pad 4: unconnected-(U2-Pad4) -> UART_RX
- U2 pad 5: unconnected-(U2-Pad5) -> UART_TX
Routing:
- net UART_RX: track 0.00 -> 78.2 mm
- net DimmerPWM: track 0.00 -> 68.6 mm
- net UART_TX: track 0.00 -> 67.5 mm
- net GND: track 0.00 -> 63.4 mm
- net 5V: track 0.00 -> 43.4 mm
- net PressureSCL: track 0.00 -> 42.4 mm
- net Display_SDA: track 0.00 -> 39.6 mm
- net Heater: track 0.00 -> 37.5 mm
- net Display_SCL: track 0.00 -> 36.8 mm
- net PressureSDA: track 0.00 -> 36.5 mm
- net Rotary_Button: track 0.00 -> 35.9 mm
- net Rotary_DT: track 0.00 -> 29.5 mm
- net Rotary_CLK: track 0.00 -> 26.6 mm
- net GroupHeadSolenoid: track 0.00 -> 16.6 mm
- net MAX6675_SO: track 0.00 -> 14.3 mm
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Other:
- board outline added: 86.4 x 66 mm

Commit message: working on max6675
Parts:
- added U3: MAX6675, OpenCoffeePartsFootprint:MAX6675, F.Cu at (185.4, 81.3)
Changed lines of the file:
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@@
   (net 82 "5V")
   (net 83 "GND")
+  (net 84 "unconnected-(U3-Pad2)")
+  (net 85 "unconnected-(U3-Pad3)")
+  (net 86 "unconnected-(U3-Pad4)")
+  (net 87 "unconnected-(U3-Pad5)")
+  (net 88 "unconnected-(U3-Pad6)")
+  (net 89 "unconnected-(U3-Pad7)")
+  (net 90 "unconnected-(U3-Pad8)")
   (footprint "Connector_Molex:Molex_KK-254_AE-6410-03A_1x03_P2.54mm_Vertical" (layer "F.Cu")
     (at 121.92 99.06)
@@
     )
   )
+  (footprint "OpenCoffeePartsFootprint:MAX6675" (layer "F.Cu")
+    (at 185.42 81.28)
+    (property "Sheetfile" "OpenCoffeePCB.kicad_sch")
+    (property "Sheetname" "")
+    (attr smd)
+    (fp_text reference "U3" (at 0 7.62 unlocked) (layer "F.SilkS")
+      (effects (font (size 1 1) (thickness 0.15)))
+    )
+    (fp_text value "MAX6675" (at 0 1 unlocked) (layer "F.Fab")
+      (effects (font (size 1 1) (thickness 0.15)))
+    )
+    (fp_text user "${REFERENCE}" (at 0 15.24) (layer "F.Fab")
+      (effects (font (size 1 1) (thickness 0.15)))
+    )
+    (fp_line (start 5.08 2.54) (end -5.08 2.54) (layer "F.CrtYd") (width 0.05))
+    (fp_line (start 5.08 12.7) (end 5.08 2.54) (layer "F.CrtYd") (width 0.05))
+    (fp_line (start -5.08 2.54) (end -5.08 12.7) (layer "F.CrtYd") (width 0.05))
+    (fp_line (start -5.08 12.7) (end 5.08 12.7) (layer "F.CrtYd") (width 0.05))
+    (fp_line (start -2.54 5.08) (end 2.54 5.08) (layer "F.Fab") (width 0.1))
+    (fp_line (start -2.54 10.16) (end -2.54 5.08) (layer "F.Fab") (width 0.1))
+    (fp_line (start 2.54 5.08) (end 2.54 10.16) (layer "F.Fab") (width 0.1))
+    (fp_line (start 2.54 10.16) (end -2.54 10.16) (layer "F.Fab") (width 0.1))
+    (pad "1" smd roundrect (at -1.915 4.915 90) (size 1.95 0.6) (layers "F.Cu" "F.Paste" "F.Mask") (roundrect_rratio 0.25)
+      (net 83 "GND") (pinfunction "GND") (pintype "input"))
+    (pad "2" smd roundrect (at -0.635 4.915 90) (size 1.6 0.6) (layers "F.Cu" "F.Paste" "F.Mask") (roundrect_rratio 0.25)
+      (net 84 "unconnected-(U3-Pad2)") (pinfunction "T-") (pintype "input"))
+    (pad "3" smd roundrect (at 0.635 4.915 90) (size 1.6 0.6) (layers "F.Cu" "F.Paste" "F.Mask") (roundrect_rratio 0.25)
+      (net 85 "unconnected-(U3-Pad3)") (pinfunction "T+") (pintype "input"))
+    (pad "4" smd roundrect (at 1.905 4.915 90) (size 1.6 0.6) (layers "F.Cu" "F.Paste" "F.Mask") (roundrect_rratio 0.25)
+      (net 86 "unconnected-(U3-Pad4)") (pinfunction "VCC") (pintype "input"))
+    (pad "5" smd roundrect (at 1.905 10.325 90) (size 1.6 0.6) (layers "F.Cu" "F.Paste" "F.Mask") (roundrect_rratio 0.25)
+      (net 87 "unconnected-(U3-Pad5)") (pinfunction "SCK") (pintype "input"))
+    (pad "6" smd roundrect (at 0.635 10.325 90) (size 1.6 0.6) (layers "F.Cu" "F.Paste" "F.Mask") (roundrect_rratio 0.25)
+      (net 88 "unconnected-(U3-Pad6)") (pinfunction "CS") (pintype "input"))
+    (pad "7" smd roundrect (at -0.635 10.325 90) (size 1.6 0.6) (layers "F.Cu" "F.Paste" "F.Mask") (roundrect_rratio 0.25)
+      (net 89 "unconnected-(U3-Pad7)") (pinfunction "SO") (pintype "input"))
+    (pad "8" smd roundrect (at -1.905 10.325 90) (size 1.6 0.6) (layers "F.Cu" "F.Paste" "F.Mask") (roundrect_rratio 0.25)
+      (net 90 "unconnected-(U3-Pad8)") (pinfunction "NC") (pintype "input"))
+  )
   (footprint "Connector_Molex:Molex_KK-254_AE-6410-03A_1x03_P2.54mm_Vertical" (layer "F.Cu")

Commit message: working on pcb
Parts:
- added C1: 0.1uF, Capacitor_SMD:C_0805_2012Metric, F.Cu at (168.6, 48.3)
- added J9: Conn_01x02_Male, Connector_Molex:Molex_KK-254_AE-6410-02A_1x02_P2.54mm_Vertical, F.Cu at (172.7, 38.1)
- J1, J2, J3, J4, J5: footprint Connector_Molex:Molex_KK-254_AE-6410-03A_1x03_P2.54mm_Vertical -> Connector_Molex:Molex_KK-254_AE-6410-02A_1x02_P2.54mm_Vertical
- moved J3 69.3 mm to (154.9, 38.1)
- moved J6 67.1 mm to (162.6, 38.1)
- moved J1 65.5 mm to (149.9, 38.1), turned to 180 degrees
- moved J5 50.8 mm to (142.2, 38.1), turned to 180 degrees
- moved J7 38.1 mm to (134.6, 38.1), turned to 180 degrees
- moved U3 36.3 mm to (170.8, 48.1)
- moved U2 35.3 mm to (134.6, 83.8), turned to 90 degrees
- moved J2 21.8 mm to (124.5, 38.1), turned to 180 degrees
- moved U1 8.98 mm to (135.9, 57.1), turned to 90 degrees
- moved J4 8.03 mm to (114.3, 38.1), turned to 180 degrees
- moved J8 7.11 mm to (188.6, 47.0)
Connections:
- U1 pad 36: 5V -> unconnected-(U1-3V3-Pad36)
- U1 pad 39: unconnected-(U1-Pad39) -> 5V
- U2 pad 36: 5V -> unconnected-(U2-3V3-Pad36)
- U2 pad 39: unconnected-(U2-Pad39) -> 5V
- U3 pad 2: unconnected-(U3-Pad2) -> T-
- U3 pad 3: unconnected-(U3-Pad3) -> T+
- U3 pad 4: unconnected-(U3-Pad4) -> 5V
- U3 pad 5: unconnected-(U3-Pad5) -> MAX6675_SCK
- U3 pad 6: unconnected-(U3-Pad6) -> MAX6675_CS
- U3 pad 7: unconnected-(U3-Pad7) -> MAX6675_SO
Routing:
- net UART_RX: track 78.2 -> 0.00 mm
- net DimmerPWM: track 68.6 -> 0.00 mm
- net UART_TX: track 67.5 -> 0.00 mm
- net GND: track 63.4 -> 0.00 mm
- net 5V: track 43.4 -> 0.00 mm
- net PressureSCL: track 42.4 -> 0.00 mm
- net Display_SDA: track 39.6 -> 0.00 mm
- net Heater: track 37.5 -> 0.00 mm
- net Display_SCL: track 36.8 -> 0.00 mm
- net PressureSDA: track 36.5 -> 0.00 mm
- net Rotary_Button: track 35.9 -> 0.00 mm
- net Rotary_DT: track 29.5 -> 0.00 mm
- net Rotary_CLK: track 26.6 -> 0.00 mm
- net GroupHeadSolenoid: track 16.6 -> 0.00 mm
- net MAX6675_SO: track 14.3 -> 0.00 mm
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
Commit message: making PCB
Parts:
- added J10: Conn_01x02_Male, Connector_Molex:Molex_KK-254_AE-6410-02A_1x02_P2.54mm_Vertical, F.Cu at (176.5, 38.1)
- moved J7 8.89 mm to (125.7, 38.1), turned to 0 degrees
- moved J1 6.35 mm to (143.5, 38.1), turned to 0 degrees
- moved J5 6.35 mm to (135.9, 38.1), turned to 0 degrees
- moved J2 5.08 mm to (119.4, 38.1), turned to 0 degrees
- moved J3 3.81 mm to (151.1, 38.1)
- moved J6 3.81 mm to (158.8, 38.1)
- moved J9 3.81 mm to (168.9, 38.1)
- moved J4 2.54 mm to (111.8, 38.1), turned to 0 degrees
- moved C1 1.27 mm to (169.9, 48.3)
Connections:
- J4 pad 1: UART_RX -> UART_RX_W
- J4 pad 2: UART_TX -> UART_TX_W
- U1 pad 13: unconnected-(U1-GND-Pad13) -> GND
- U1 pad 18: unconnected-(U1-GND-Pad18) -> GND
- U1 pad 23: unconnected-(U1-GND-Pad23) -> GND
- U1 pad 42: unconnected-(U1-GND-Pad42) -> GND
- U2 pad 13: unconnected-(U2-GND-Pad13) -> GND
- U2 pad 18: unconnected-(U2-GND-Pad18) -> GND
- U2 pad 23: unconnected-(U2-GND-Pad23) -> GND
- U2 pad 3: unconnected-(U2-GND-Pad3) -> GND
- U2 pad 33: unconnected-(U2-AGND-Pad33) -> GND
- U2 pad 38: unconnected-(U2-GND-Pad38) -> GND
- U2 pad 4: UART_RX -> UART_RX_W
- U2 pad 5: UART_TX -> UART_TX_W
- U2 pad 8: unconnected-(U2-GND-Pad8) -> GND
Routing:
- net GND: track 0.00 -> 211.2 mm
- net 5V: track 0.00 -> 110.6 mm, vias 0 -> 1
- net MAX6675_SCK: track 0.00 -> 63.1 mm
- net UART_TX: track 0.00 -> 60.1 mm
- net UART_TX_W: track 0.00 -> 57.9 mm
- net UART_RX_W: track 0.00 -> 57.2 mm
- net UART_RX: track 0.00 -> 56.5 mm
- net GroupHeadSolenoid: track 0.00 -> 52.3 mm
- net Display_SDA: track 0.00 -> 48.8 mm
- net Rotary_DT: track 0.00 -> 47.2 mm
- net Rotary_Button: track 0.00 -> 45.4 mm
- net DimmerPWM: track 0.00 -> 36.4 mm
- net Display_SCL: track 0.00 -> 34.8 mm
- net Rotary_CLK: track 0.00 -> 30.6 mm
- net MAX6675_SO: track 0.00 -> 30.0 mm, vias 0 -> 1
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
Commit message: part
Parts:
- C1: value 0.1uF -> C
Routing:
- net T-: track 15.4 -> 37.9 mm
- net GroupHeadSolenoid: track 52.3 -> 33.7 mm
- net 5V: track 110.6 -> 121.7 mm, vias 1 -> 0
- net Rotary_DT: track 47.2 -> 38.3 mm
- net MAX6675_SCK: track 63.1 -> 54.3 mm
- net Display_SDA: track 48.8 -> 41.7 mm
- net GND: track 211.2 -> 217.1 mm
- net T+: track 15.1 -> 20.4 mm, vias 0 -> 1
- net UART_TX: track 60.1 -> 65.2 mm
- net DimmerPWM: track 36.4 -> 38.8 mm
- net MAX6675_CS: track 28.3 -> 26.0 mm, vias 1 -> 0
- net MAX6675_SO: track 30.0 -> 27.9 mm, vias 1 -> 0
- net UART_TX_W: track 57.9 -> 59.0 mm
- net UART_RX_W: track 57.2 -> 58.2 mm
