File: OpenCoffee_PCB/OpenCoffeePCB/OpenCoffeePCB.kicad_pcb (KiCad board)
At the start: 2 copper layers, 86.4 x 66 mm, 14 parts, among them J1 Conn_01x02_Male, J10 Conn_01x02_Male, J2 Conn_01x02_Male, J3 Conn_01x02_Male, J4 Conn_01x02_Male, J5 Conn_01x02_Male, J6 Conn_01x03_Male, J7 Conn_01x03_Male, J8 Barrel_Jack_Switch, J9 Conn_01x02_Male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

Commit message: added RP2040 from https://datasheets.raspberrypi.com/rp2040/Minimal-KiCAD.zip?_gl=1*n2lfxt*_ga*MTI3MDcyNzk1MS4xNjg5NTU4NDUx*_ga_22FD70LWDS*MTY4OTU1ODQ1Mi4xLjEuMTY4OTU1OTgzMS4wLjAuMA..
Parts:
- added C10: 100n, Capacitor_SMD:C_0402_1005Metric, F.Cu at (226.1, 81.9)
- added C11: 1u, Capacitor_SMD:C_0402_1005Metric, F.Cu at (228.9, 70.1)
- added C12: 100n, Capacitor_SMD:C_0402_1005Metric, F.Cu at (228.9, 72.1)
- added C13: 100n, Capacitor_SMD:C_0402_1005Metric, F.Cu at (228.9, 74.0)
- added C14: 100n, Capacitor_SMD:C_0402_1005Metric, F.Cu at (228.9, 76.0)
- added C15: 100n, Capacitor_SMD:C_0402_1005Metric, F.Cu at (228.9, 78.0)
- added C16: 100n, Capacitor_SMD:C_0402_1005Metric, F.Cu at (228.9, 80.0)
- added C17: 100n, Capacitor_SMD:C_0402_1005Metric, F.Cu at (228.9, 81.9)
- added C2: 10u, Capacitor_SMD:C_0805_2012Metric, F.Cu at (235.4, 85.6)
- added C3: 10u, Capacitor_SMD:C_0805_2012Metric, F.Cu at (235.4, 88.7)
- added C4: 100n, Capacitor_SMD:C_0402_1005Metric, F.Cu at (226.1, 70.1)
- added C5: 27p, Capacitor_SMD:C_0402_1005Metric, F.Cu at (226.1, 72.1)
- added C6: 27p, Capacitor_SMD:C_0402_1005Metric, F.Cu at (226.1, 74.0)
- added C7: 100n, Capacitor_SMD:C_0402_1005Metric, F.Cu at (226.1, 76.0)
- added C8: 100n, Capacitor_SMD:C_0402_1005Metric, F.Cu at (226.1, 78.0)
- added C9: 1u, Capacitor_SMD:C_0402_1005Metric, F.Cu at (226.1, 80.0)
- added J11: USB_B_Micro, RP2040_minimal:USB_Micro-B_Amphenol_10103594-0001LF_Horizontal_modified, F.Cu at (223.5, 53.3)
- added J12: Conn_01x02, Connector_PinHeader_2.54mm:PinHeader_1x02_P2.54mm_Vertical, F.Cu at (245.1, 68.6)
- added R1: 1k, Capacitor_SMD:C_0402_1005Metric, F.Cu at (231.8, 70.1)
- added R2: DNF, Capacitor_SMD:C_0402_1005Metric, F.Cu at (231.8, 72.1)
- added R3: 1k, Capacitor_SMD:C_0402_1005Metric, F.Cu at (231.8, 74.0)
- added R4: 27, Capacitor_SMD:C_0402_1005Metric, F.Cu at (231.8, 76.0)
- added R5: 27, Capacitor_SMD:C_0402_1005Metric, F.Cu at (231.8, 78.0)
- added U4: NCP1117-3.3_SOT223, Package_TO_SOT_SMD:SOT-223-3_TabPin2, F.Cu at (261.0, 81.3)
- added U5: W25Q128JVS, Package_SO:SOIC-8_5.23x5.23mm_P1.27mm, F.Cu at (264.2, 63.5)
- added U6: RP2040, RP2040_minimal:RP2040-QFN-56, F.Cu at (243.5, 54.5)
- added Y1: ABLS-12.000MHZ-B4-T, RP2040_minimal:Crystal_SMD_HC49-US, F.Cu at (244.5, 31.8)
